File: LabSupply 2025-2026.kicad_sch (KiCad schematic)
At the start: 1 part

Commit message: upload
Parts:
- added A1: RaspberryPi_Pico, PICO, symbol MCU_Module:RaspberryPi_Pico
- added C1: 100n, Capacitor_SMD:C_0805_2012Metric, symbol Device:C
- added C10, C14, C15, C17, C7: 100p, Capacitor_SMD:C_0805_2012Metric, symbol Device:C
- added C11, C12, C13, C16, C18: NC, Capacitor_SMD:C_0805_2012Metric, symbol Device:C
- added C2, C4, C5, C8: 1u, Capacitor_SMD:C_1206_3216Metric_Pad1.33x1.80mm_HandSolder, symbol Device:C
- added C3, C6: 220u, Capacitor_THT:CP_Radial_D8.0mm_P5.00mm, symbol Device:C_Polarized
- added C9: 22u, Capacitor_THT:CP_Radial_D8.0mm_P5.00mm, symbol Device:C_Polarized
- added D1, D2, D3, D4, D6: LL4148, Diode_SMD:D_SOD-123, symbol Diode:LL4148
- added D5: D_Schottky_AKA, Package_TO_SOT_SMD:TO-252-2, symbol Device:D_Schottky_AKA
- added D7: 2v4, Diode_SMD:D_MiniMELF, symbol Device:D_Zener
- added J1: Screw_Terminal_01x02, TerminalBlock_MetzConnect:TerminalBlock_MetzConnect_Type055_RT01502HDWU_1x02_P5.00mm_Horizontal, symbol Connector:Screw_Terminal_01x02
- added JP1: SolderJumper_3_Bridged12, Jumper:SolderJumper-3_P1.3mm_Bridged12_RoundedPad1.0x1.5mm_NumberLabels, symbol Jumper:SolderJumper_3_Bridged12
- added L1: L, Inductor_SMD:L_Bourns-SRU1028_10.0x10.0mm, symbol Device:L
- added Q1, Q11, Q12, Q14, Q2, Q3: 2N7002K, Package_TO_SOT_SMD:SOT-23, symbol Transistor_FET:2N7002K
- added Q10, Q13, Q15: BUZ11, Package_TO_SOT_THT:TO-220-3_Vertical, symbol Transistor_FET:BUZ11
- added Q5, Q8: BC807, Package_TO_SOT_SMD:SOT-23, symbol Transistor_BJT:BC807
- added Q7: TIP41B, Package_TO_SOT_THT:TO-220-3_Vertical, symbol Transistor_BJT:TIP41B
- added Q9: BC817, Package_TO_SOT_SMD:SOT-23, symbol Transistor_BJT:BC817
- added R10, R11, R13, R14, R17, R21, R22, R26, R31, R32, R33, R35, R37, R38, R41, R42, R45, R46, R49, R50, R9: 2k2, Resistor_SMD:R_0805_2012Metric, symbol Device:R
- added R12, R20, R7: 1k2, Resistor_SMD:R_0805_2012Metric, symbol Device:R
- added R15, R25, R27, R34, R36, R44: NC, Resistor_SMD:R_0805_2012Metric, symbol Device:R
- added R16, R8: 33k, Resistor_SMD:R_0805_2012Metric, symbol Device:R
- added R18, R19, R28, R43: 50m, Resistor_SMD:R_2512_6332Metric_Pad1.40x3.35mm_HandSolder, symbol Device:R
- added R2, R3, R4, R5, R6: 10k, Resistor_SMD:R_0805_2012Metric, symbol Device:R
- added R23, R24, R52, R53, R54: 39k, Resistor_SMD:R_0805_2012Metric, symbol Device:R
- added R29, R30, R39, R40, R47, R48, R55, R57: 47k, Resistor_SMD:R_0805_2012Metric, symbol Device:R
- added R51: 500m, Resistor_SMD:R_2512_6332Metric_Pad1.40x3.35mm_HandSolder, symbol Device:R
- added R56, R58: 4k7, Resistor_SMD:R_0805_2012Metric, symbol Device:R
- added U1: MCP4728, Package_SO:MSOP-10_3x3mm_P0.5mm, symbol Analog_DAC:MCP4728
- added U2: APE1707H-HF, Package_TO_SOT_SMD:TO-252-5_TabPin3, symbol Regulator_Switching:APE1707H-HF
- added U3, U5, U6: LM324, Package_SO:SOIC-14_3.9x8.7mm_P1.27mm, symbol Amplifier_Operational:LM324
- added U4, U7: 74LVC1G3157, Package_TO_SOT_SMD:SOT-23-6_Handsoldering, symbol 74xGxx:74LVC1G3157
- R1: value R -> 10k; footprint Resistor_SMD:R_0603_1608Metric_Pad0.98x0.95mm_HandSolder -> Resistor_SMD:R_0805_2012Metric
Connections:
- net +3V3: now reaches R1.1
- net +3V3: now also Q1.1 (G), Q2.1 (G), Q3.1 (G), R3.1, R5.1, U4.5 (VCC), U7.5 (VCC)
- net SCL: now reaches R1.2
- net SCL: now also Q1.2 (S)
- new net: R52.2, R54.1, U6.7
- new net: D7.1 (K), R54.2, U4.3, U7.3
- new net: R38.2, R39.1, U5.14
- new net: R39.2, R42.1, U5.13 (-)
- new net: JP1.2 (C), R12.2
- new net: C17.1, C18.1, R45.1, U6.8
- new net: C17.2, R44.2, R46.1, U6.9 (-)
- new net: D2.2 (A), D3.1 (K)
- new net: C2.1, C6.1, D3.2 (A), D4.1 (K), L1.2, Q7.2 (C), Q8.2 (E), R11.1, R8.1
- new net: C7.2, R15.2, R16.2, R17.1, U3.6 (-)
- new net: Q10.3 (S), R28.1, R31.2
- new net: C10.2, C12.1, R25.2, R26.1, U3.13 (-)
- new net: D5.2 (K), L1.1, U2.2 (SW)
- new net: R7.1, R8.2, R9.1, U2.4 (FB)
- new net: C18.2, R44.1
- new net: Q1.3 (D), R2.2, U1.2 (SCL)
- new net: R47.2, R50.1, U6.13 (-)
- new net: C13.1, C14.1, R35.1, U5.7
- new net: C14.2, R33.1, R34.2, U5.6 (-)
- new net: Q8.1 (B), Q9.3 (C), R11.2
- new net: Q7.1 (B), Q8.3 (C)
- new net: Q2.3 (D), R4.2, U1.3 (SDA)
- new net: U5.10 (+), U5.5 (+), U7.4
- new net: C13.2, R34.1
- new net: Q12.3 (D), Q13.1 (G), R37.2
- new net: Q13.3 (S), R41.2, R43.1
- new net: R40.2, R41.1, U5.12 (+)
- new net: R13.2, R14.1, R15.1, U3.7
- new net: R21.1, R23.2, U3.10 (+)
- new net: R22.1, R24.2, U3.9 (-)
- new net: C15.1, C16.1, R37.1, U5.8
- new net: C16.2, R36.1
- new net: R29.2, R32.1, U5.2 (-)
- new net: D6.2 (A), Q9.1 (B), R13.1, R53.1
- new net: R52.1, R53.2, U6.6 (-)
- new net: C15.2, R36.2, R38.1, U5.9 (-)
- new net: Q10.1 (G), Q11.3 (D), R35.2
- new net: D1.2 (A), D2.1 (K)
- new net: D4.2 (A), Q5.1 (B), R10.1
- new net: Q15.3 (S), R49.2, R51.1
- new net: R48.2, R49.1, U6.12 (+)
- new net: R30.2, R31.1, U5.3 (+)
- new net: D6.1 (K), R20.1
- new net: C10.1, C11.1, R20.2, U3.14
- new net: Q14.3 (D), Q15.1 (G), R45.2
- new net: U4.4, U6.10 (+)
- new net: C7.1, R14.2
- new net: D1.1 (K), Q5.2 (E)
- new net: C12.2, R27.1
- new net: Q3.3 (D), R6.2, U1.4 (~{LDAC})
- new net: C11.2, R25.1
- new net: Q5.3 (C), R9.2
- new net: R10.2, U3.1, U3.2 (-)
- new net: A1.13 (GND), A1.18 (GND), A1.23 (GND), A1.28 (GND), A1.3 (GND), A1.38 (GND), A1.8 (GND)
- new net: Q9.2 (E), R12.1
- new net +12V: U5.4 (V+), U6.4 (V+)
- new net +24V: C3.1, C4.1, C5.1, R57.1, U2.1 (VCC), U3.4 (V+)
- new net +5V: R2.1, R4.1, R6.1
- new net +5VA: U1.1 (VDD)
- new net -3V3: JP1.3 (B), U3.11 (V-), U5.11 (V-), U6.11 (V-), U6.2 (-)
- new net GND: C2.2, C3.2, C4.2, C5.2, C6.2, D5.1 (A), D5.3 (A), D7.2 (A), JP1.1 (A), Q11.2 (S), Q12.2 (S), Q14.2 (S), R17.2, R18.2, R19.2, R22.2, R23.1, R30.1, R40.1, R48.1, R56.2, R58.2, R7.2, U1.10 (VSS), U2.3 (VSS), U2.5 (~{EN}), U4.2 (GND), U6.3 (+), U6.5 (+), U7.2 (GND)
- new net H-Iref: U1.8 (VOUTC), U7.1
- new net HighCurrent-enable: Q11.1 (G), Q12.1 (G)
- new net HighCurrent-measured: R29.1, R33.2, U5.1
- new net HighCurrentSwitch: U7.6
- new net Iref: U1.7 (VOUTB), U3.12 (+)
- new net L-Iref: U1.9 (VOUTD), U4.1
- new net LDAC: Q3.2 (S), R5.2
- new net LowCurrent-enable: Q14.1 (G)
- new net LowCurrent-measured: R46.2, R47.1, U6.14
- new net LowCurrentSwitch: U4.6
- new net SDA: Q2.2 (S), R3.2
- new net Vin-measured: R57.2, R58.1
- new net Vout+: C8.1, C9.1, J1.1 (Pin_1), Q10.2 (D), Q13.2 (D), Q15.2 (D), Q7.3 (E), R16.1, R55.1, U3.3 (+)
- new net Vout-: C8.2, C9.2, J1.2 (Pin_2), R18.1, R19.1, R21.2, R28.2, R32.2, R42.2, R43.2, R50.2, R51.2
- new net Vout-measured: R55.2, R56.1
- new net Vref: U1.6 (VOUTA), U3.5 (+)
- new net current-measured: R24.1, R26.2, R27.2, U3.8
- no-connect marks 0 -> 2
Other:
- note added: "47k"
- note added: "OR LM1501BGR-ADJ"
- note added: "electronic load"
- note added: "might need smaller resistor to start properly"
- note added: "power supply"

Commit message: added buck power supplies
Parts:
- removed U3: LM324, Package_SO:SOIC-14_3.9x8.7mm_P1.27mm, symbol Amplifier_Operational:LM324
- added 12V, 15V, 5V, 5Va: TestPoint_Probe, TestPoint:TestPoint_Pad_D2.0mm, symbol Connector:TestPoint_Probe
- added C19, C20, C21, C22, C23, C24, C33, C34, C35: 100n, Capacitor_SMD:C_0805_2012Metric, symbol Device:C
- added C25, C28, C29, C31: 1u, Capacitor_SMD:C_1206_3216Metric_Pad1.33x1.80mm_HandSolder, symbol Device:C
- added C26: 100p, Capacitor_SMD:C_0805_2012Metric, symbol Device:C
- added C27, C32: 220u, Capacitor_THT:CP_Radial_D8.0mm_P5.00mm, symbol Device:C_Polarized
- added C30: 330p, Capacitor_SMD:C_0805_2012Metric, symbol Device:C
- added D10: LL4148, Diode_SMD:D_SOD-123, symbol Diode:LL4148
- added D11, D12: D_Schottky, Diode_SMD:D_SMA, symbol Device:D_Schottky
- added D8, D9: D_Schottky_AKA, Package_TO_SOT_SMD:TO-252-2, symbol Device:D_Schottky_AKA
- added JP2, JP3: SolderJumper_2_Open, Jumper:SolderJumper-2_P1.3mm_Open_RoundedPad1.0x1.5mm, symbol Jumper:SolderJumper_2_Open
- added L2: 220u, Inductor_SMD:L_Bourns-SRU1028_10.0x10.0mm, symbol Device:L
- added L3: 470u, Inductor_SMD:L_Bourns-SRU1028_10.0x10.0mm, symbol Device:L
- added R59, R60: 2k2, Resistor_SMD:R_0805_2012Metric, symbol Device:R
- added R61: 1M, Resistor_SMD:R_0805_2012Metric, symbol Device:R
- added R62, R65: 1, Resistor_SMD:R_0805_2012Metric, symbol Device:R
- added R63: 3k, Resistor_SMD:R_0805_2012Metric, symbol Device:R
- added R64, R67: 1k, Resistor_SMD:R_0805_2012Metric, symbol Device:R
- added R66: 11k, Resistor_SMD:R_0805_2012Metric, symbol Device:R
- added U10, U8, U9: RC4580, Package_SO:SOIC-8_3.9x4.9mm_P1.27mm, symbol Amplifier_Operational:RC4580
- added U11, U3: MC34063AD, Package_SO:SOIC-8_3.9x4.9mm_P1.27mm, symbol Regulator_Switching:MC34063AD
- added U12: L78L12_SO8, Package_SO:SOIC-8_3.9x4.9mm_P1.27mm, symbol Regulator_Linear:L78L12_SO8
- added U13: L78L05_SO8, Package_SO:SOIC-8_3.9x4.9mm_P1.27mm, symbol Regulator_Linear:L78L05_SO8
- C11, C12, C13, C16, C18, R25, R27, R34, R36, R44: now not fitted
- R15: value NC -> 47k; now not fitted
Connections:
- net +12V: now also 12V.1, C19.2, C20.2, C22.2, C23.2, C33.2, R61.1, U12.1 (OUT), U13.8 (IN), U8.8 (V+), U9.8 (V+)
- net +5V: now also 5V.1, C27.1, C28.1, D10.2 (A), L2.2, R63.2
- net +5VA: now also 5Va.1, C24.2, C34.2, D10.1 (K), U13.1 (OUT)
- net -3V3: now also C19.1, C20.1, C21.1, C22.1, C23.1, U10.4 (V-), U8.4 (V-), U9.4 (V-); no longer U6.2 (-)
- net GND: now also C24.1, C25.2, C26.1, C27.2, C28.2, C29.2, C30.1, C31.2, C32.2, C33.1, C35.1, D11.2 (A), D12.2 (A), R64.1, R67.1, U10.5 (+), U11.4 (GND), U12.2 (GND), U12.3 (GND), U12.6 (GND), U12.7 (GND), U13.2 (GND), U13.3 (GND), U13.6 (GND), U13.7 (GND), U3.4 (GND)
- net Iref: now also U9.3 (+)
- net Vout+: now also D8.2 (K), JP2.2 (B), R59.1; no longer Q7.3 (E)
- net Vref: now also U8.3 (+)
- net current-measured: now also U9.7
- net at C2.1, C6.1, D3.2 (A)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: now also D9.2 (K)
- net at R16.2, R17.1: now also U8.5 (+); no longer C7.2, R15.2
- net at C10.2, C12.1, R25.2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: now also U9.2 (-)
- net at R13.2, R14.1, R15.1: now also U8.1
- net at R21.1, R23.2: now also R61.2, U9.5 (+)
- net at R22.1, R24.2: now also U9.6 (-)
- net at C10.1, C11.1, R20.2: now also U9.1
- net at U6.1: now also U6.2 (-)
- net at R10.2: now also U10.1, U10.2 (-)
- net +24V renamed +28V
- net +28V: now also C21.2, C25.1, C29.1, JP3.1 (A), R62.2, R65.2, U10.8 (V+), U11.6 (Vin), U3.6 (Vin)
- new net: D11.1 (K), L2.1, U3.2 (SwE)
- new net: R63.1, R64.2, U3.5 (Vfb)
- new net: R66.1, R67.2, U11.5 (Vfb)
- new net: C7.2, R15.2, U8.2 (-), U8.6 (-), U8.7
- new net: D8.1 (A), D8.3 (A), D9.1 (A), D9.3 (A), JP2.1 (A), Q7.3 (E), R60.1
- new net: R62.1, U3.1 (SwC), U3.7 (Ipk), U3.8 (DC)
- new net: D12.1 (K), L3.1, U11.2 (SwE)
- new net: R59.2, R60.2, U10.3 (+)
- new net: C26.2, U3.3 (TC)
- new net: R65.1, U11.1 (SwC), U11.7 (Ipk), U11.8 (DC)
- new net: C30.2, U11.3 (TC)
- new net: U10.6 (-), U10.7
- new net +15V: 15V.1, C31.1, C32.1, C35.2, JP3.2 (B), L3.2, R66.2, U12.8 (IN)
- no-connect marks 2 -> 1
Other:
- note added: "15v buck converter supply"
- note added: "5v buck converter supply"
- note added: "65kHz"
- note added: "75kHz"
- note added: "DAC for controlling power supply"
- note added: "Iout = 150mA"
- note added: "analog power section"
- note added: "level shifter"
- note added: "min 300mA"
- note added: "switching preregulator"
- note removed: "47k"
- note removed: "power supply"
- moved on the sheet: C4, C5, D1, D2, D3, D4, Q1, Q2, Q3, Q5, R1, R10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

Commit message: almost complete schematics
Parts:
- removed C1: 100n, Capacitor_SMD:C_0805_2012Metric, symbol Device:C
- added -3v3, -5v, ADC-free: TestPoint_Probe, TestPoint:TestPoint_Pad_D2.0mm, symbol Connector:TestPoint_Probe
- added C36, C38, C45, C46, C47, C48, C49, C50: 1u, Capacitor_SMD:C_1206_3216Metric_Pad1.33x1.80mm_HandSolder, symbol Device:C
- added C37: 100p, Capacitor_SMD:C_0805_2012Metric, symbol Device:C
- added C39: 220u, Capacitor_THT:CP_Radial_D8.0mm_P5.00mm, symbol Device:C_Polarized
- added C40, C51, C52, C53: 100n, Capacitor_SMD:C_0805_2012Metric, symbol Device:C
- added C41: 1u, Capacitor_SMD:C_0805_2012Metric, symbol Device:C
- added C42, C43, C44: 10n, Capacitor_SMD:C_2220_5750Metric, symbol Device:C
- added C54, C57: 100u, Capacitor_THT:CP_Radial_D6.3mm_P2.50mm, symbol Device:C_Polarized
- added C55, C56: 4u7, Capacitor_SMD:C_0805_2012Metric_Pad1.18x1.45mm_HandSolder, symbol Device:C
- added C58, C59: 10n, Capacitor_SMD:C_0805_2012Metric, symbol Device:C
- added D13, D15: D_Schottky, Diode_SMD:D_SMA, symbol Device:D_Schottky
- added D14: 1N62xxA, Diode_THT:D_DO-201AE_P15.24mm_Horizontal, symbol Diode:1N62xxA
- added D16, D18, D19: LL4148, Diode_SMD:D_SOD-123, symbol Diode:LL4148
- added D17: 3v9, Diode_SMD:D_SMB-SMC_Universal_Handsoldering, symbol Device:D_Zener
- added FL1: Choke_CommonMode_PulseElectronics_PH9455x156NL, Inductor_THT:L_CommonMode_PulseElectronics_PH9455xxx6NL_2, symbol Filter:Choke_CommonMode_PulseElectronics_PH9455x156NL
- added H1: MountingHole_Pad, MountingHole:MountingHole_3.2mm_M3_ISO7380_Pad, symbol Mechanical:MountingHole_Pad
- added J2: Conn_02x17_Odd_Even, Connector_IDC:IDC-Header_2x17_P2.54mm_Latch6.5mm_Vertical, symbol Connector_Generic:Conn_02x17_Odd_Even
- added J3: Screw_Terminal_01x02, TerminalBlock_MetzConnect:TerminalBlock_MetzConnect_Type055_RT01502HDWU_1x02_P5.00mm_Horizontal, symbol Connector:Screw_Terminal_01x02
- added L4: 220u, Inductor_SMD:L_Bourns-SRU1028_10.0x10.0mm, symbol Device:L
- added LS1: Speaker, Buzzer_Beeper:MagneticBuzzer_ProjectsUnlimited_AI-4228-TWT-R, symbol Device:Speaker
- added Q16: BD136, Package_TO_SOT_THT:TO-126-3_Vertical, symbol Transistor_BJT:BD136
- added Q4: 2N7002K, Package_TO_SOT_SMD:SOT-23, symbol Transistor_FET:2N7002K
- added Q6: BD139, Package_TO_SOT_THT:TO-126-3_Vertical, symbol Transistor_BJT:BD139
- added R68: 1, Resistor_SMD:R_0805_2012Metric, symbol Device:R
- added R69, R74: 1M, Resistor_SMD:R_1206_3216Metric, symbol Device:R
- added R70, R73: 3k, Resistor_SMD:R_0805_2012Metric, symbol Device:R
- added R71, R72, R75: 1k, Resistor_SMD:R_0805_2012Metric, symbol Device:R
- added R76, R77: 10k, Resistor_SMD:R_0805_2012Metric, symbol Device:R
- added R78, R79, R82: 33k, Resistor_SMD:R_0805_2012Metric, symbol Device:R
- added R80, R83, R84: 2k2, Resistor_SMD:R_0805_2012Metric, symbol Device:R
- added R81: 47k, Resistor_SMD:R_0805_2012Metric, symbol Device:R
- added TH1, TH2: Thermistor_NTC, Resistor_SMD:R_0805_2012Metric, symbol Device:Thermistor_NTC
- added U14: MC34063AD, Package_SO:SOIC-8_3.9x4.9mm_P1.27mm, symbol Regulator_Switching:MC34063AD
- added U15: LM337L_SO8, Package_SO:SOIC-8_3.9x4.9mm_P1.27mm, symbol Regulator_Linear:LM337L_SO8
- added U16: LM4040DBZ-3, Package_TO_SOT_SMD:SOT-23, symbol Reference_Voltage:LM4040DBZ-3
- added U17, U18, U19, U20, U21: 74LVC1G3157, Package_TO_SOT_SMD:SOT-23-6_Handsoldering, symbol 74xGxx:74LVC1G3157
- added fan: Conn_01x02_Pin, Connector_PinHeader_2.54mm:PinHeader_1x02_P2.54mm_Vertical, symbol Connector:Conn_01x02_Pin
- D10: now not fitted
Connections:
- net +12V: now also C57.1, Q6.2 (C), R78.1
- net +28V: now also C36.1, D17.1 (K), J2.18 (Pin_18), J3.2 (Pin_2), R68.2, U14.6 (Vin)
- net +3V3: now also A1.36 (3V3), U6.3 (+), J2.3 (Pin_3), J2.31 (Pin_31), J2.32 (Pin_32), J2.4 (Pin_4), R76.1, R77.1, U17.5 (VCC), U18.5 (VCC), U19.5 (VCC), U20.5 (VCC), U21.5 (VCC)
- net +5V: now also D15.2 (A), J2.1 (Pin_1), J2.2 (Pin_2), J2.33 (Pin_33), J2.34 (Pin_34)
- net -3V3: now also -3v3.1, C41.1, R72.2, U15.1 (VO)
- net GND: now also A1.13 (GND), A1.18 (GND), A1.23 (GND), A1.28 (GND), A1.3 (GND), A1.33 (AGND), A1.38 (GND), A1.8 (GND), C34.1, C36.2, C38.1, C39.1, C40.2, C41.2, C51.2, C52.1, C53.1, C57.2, C58.2, C59.2, J2.15 (Pin_15), J2.16 (Pin_16), J2.29 (Pin_29), J2.30 (Pin_30), J2.5 (Pin_5), J2.6 (Pin_6), J3.1 (Pin_1), L4.2, LS1.2, Q16.2 (C), Q4.2 (S), R70.1, R73.1, R79.2, TH1.2, TH2.2, U16.2 (A), U17.2 (GND), U18.2 (GND), U19.2 (GND), U20.2 (GND), U21.2 (GND); no longer U6.3 (+)
- net HighCurrent-enable: now also A1.26 (GPIO20)
- net LDAC: now also A1.20 (GPIO15)
- net LowCurrent-enable: now also A1.27 (GPIO21)
- net SCL: now also A1.22 (GPIO17)
- net SDA: now also A1.21 (GPIO16)
- net Vin-measured: now also U19.1
- net Vout+: now also C44.1, C49.1, C50.1, FL1.1, J2.17 (Pin_17); no longer J1.1 (Pin_1)
- net Vout-: now also C44.2, C49.2, C50.2, FL1.2, J2.19 (Pin_19), J2.20 (Pin_20); no longer J1.2 (Pin_2)
- net Vout-measured: now also U18.3
- net at U6.1: now also R80.1, R81.2; no longer U6.2 (-)
- net at A1.1 (GPIO0): now also J2.8 (Pin_8)
- net at A1.10 (GPIO7): now also J2.28 (Pin_28)
- net at A1.11 (GPIO8): now also J2.27 (Pin_27)
- net at A1.12 (GPIO9): now also J2.25 (Pin_25)
- net at A1.14 (GPIO10): now also J2.23 (Pin_23)
- net at A1.15 (GPIO11): now also J2.21 (Pin_21)
- net at A1.16 (GPIO12): now also J2.13 (Pin_13)
- net at A1.17 (GPIO13): now also J2.11 (Pin_11)
- net audio-PWM: now reaches A1.19 (GPIO14)
- net audio-PWM: now also J2.9 (Pin_9), R84.1
- net at A1.2 (GPIO1): now also J2.10 (Pin_10)
- net adc-mux2: now reaches A1.24 (GPIO18)
- net adc-mux2: now also U19.6, U21.6
- net adc-mux1: now reaches A1.25 (GPIO19)
- net adc-mux1: now also U17.6, U18.6, U20.6
- net fan: now reaches A1.29 (GPIO22)
- net fan: now also Q4.1 (G)
- net at A1.31 (GPIO26_ADC0): now also U17.4
- net at A1.32 (GPIO27_ADC1): now also U18.4
- net at A1.34 (GPIO28_ADC2): now also U20.4
- net at A1.35 (ADC_VREF): now also C51.1, R75.1, U16.1 (K)
- net at A1.39 (VSYS): now also D15.1 (K)
- net at A1.4 (GPIO2): now also J2.12 (Pin_12)
- net at A1.5 (GPIO3): now also J2.14 (Pin_14)
- net at A1.6 (GPIO4): now also J2.22 (Pin_22)
- net at A1.7 (GPIO5): now also J2.24 (Pin_24)
- net at A1.9 (GPIO6): now also J2.26 (Pin_26)
- net HighCurrent-measured renamed HighCurrent-In-measured
- net HighCurrent-In-measured: now also U20.1
- net LowCurrent-measured renamed LowCurrent-In-measured
- net LowCurrent-In-measured: now also U20.3
- net current-measured renamed Iout-measured
- net Iout-measured: now also U18.1
- new net: C59.1, R83.1, R84.2
- new net: C42.1, C45.1, C46.1, C47.1, C48.1, D14.2 (A2), FL1.3, J1.1 (Pin_1), R69.1
- new net: C43.1, C45.2, C46.2, C47.2, C48.2, D14.1 (A1), FL1.4, J1.2 (Pin_2), R74.1
- new net: C58.1, R82.1, R83.2
- new net: R70.2, R71.1, U14.5 (Vfb)
- new net: -5v.1, C37.1, C38.2, C39.2, C40.1, D13.2 (A), R71.2, U14.4 (GND), U15.2 (VI), U15.3 (VI), U15.6 (VI), U15.7 (VI)
- new net: C54.1, Q16.1 (E), Q6.1 (E)
- new net: C55.1, D18.2 (A), Q6.3 (B), R78.2
- new net: D16.1 (K), D17.2 (A), fan.2 (Pin_2)
- new net: D16.2 (A), Q4.3 (D), fan.1 (Pin_1)
- new net: C37.2, U14.3 (TC)
- new net: C55.2, C56.2, R80.2
- new net: R81.1, R82.2, U6.2 (-)
- new net: C56.1, D19.1 (K), Q16.3 (B), R79.1
- new net: D13.1 (K), L4.1, U14.2 (SwE)
- new net: R72.1, R73.2, U15.4 (ADJ)
- new net: U17.1, U19.4
- new net: U17.3, U21.4
- new net: C54.2, LS1.1
- new net: D18.1 (K), D19.2 (A)
- new net: R68.1, U14.1 (SwC), U14.7 (Ipk), U14.8 (DC)
- new net: ADC-free.1, U21.3
- new net +3.3V: R75.2
- new net Earth: C42.2, C43.2, H1.1, R69.2, R74.2
- new net temp1: C52.2, R76.2, TH1.1, U19.3
- new net temp2: C53.2, R77.2, TH2.1, U21.1
- no-connect marks 1 -> 5
Other:
- note added: "-5v buck inverting converter"
- note added: "15v buck converter"
- note added: "5v buck converter"
- note added: "Iout = 50mA"
- note added: "analog mux"
- note added: "audio power stage"
- note added: "možná pojede i s DC vazbou"
- note removed: "15v buck converter supply"
- note removed: "5v buck converter supply"
- moved on the sheet: 12V, 15V, 5V, 5Va, A1, C24, C25, C26, C27, C28, C29, C30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
